Commit message: imu added

File: description/lidar.xacro (robot description, xacro)
@@ -4,5 +4,5 @@
         <parent link="base_link"/>
         <child link="laser_link"/>
-        <origin xyz="0.1 0.0 0.09"/>
+        <origin xyz="-0.1 0.0 0.09"/>
     </joint>
     <link name="laser_link">

File: description/robot.urdf.xacro (robot description, xacro)
@@ -11,3 +11,4 @@
     </xacro:unless>
     <xacro:include filename="lidar.xacro" />
+    <xacro:include filename="imu.xacro" />
 </robot>
